File: KiCad project/ESP32-C3-02.kicad_sch (KiCad schematic)
At the start: 30 parts, among them J2 GSD090012SEU, U3 ESP32-C3-WROOM-02-H4, U4 CP2102N-Axx-xQFN20, U5 W25Q32JVSSIQ

Commit message: Fixed lots of bugs.
Parts:
- removed C10: 10u, Capacitor_SMD:C_0805_2012Metric, symbol SparkFun-Capacitor:C
- removed D6, D7: PESD5V0S1UL_315, Footprints:DIO_PESD5V0S1UL_315, symbol PESD5V0S1UL_315:PESD5V0S1UL_315
- removed R15, R16: 1K, Resistor_SMD:R_0805_2012Metric, symbol Device:R
- removed R22, R29: 50, Resistor_SMD:R_0201_0603Metric, symbol Device:R
- added C11: 1u, Capacitor_SMD:C_0805_2012Metric, symbol SparkFun-Capacitor:C
- added C8: 0.1u, Capacitor_SMD:C_0805_2012Metric, symbol SparkFun-Capacitor:C
- added R19: 10K, Resistor_SMD:R_0805_2012Metric, symbol Device:R
- added U5: USBLC6-2SC6, Package_TO_SOT_SMD:SOT-23-6, symbol Power_Protection:USBLC6-2SC6
- D6: renamed from D8; footprint SparkFun-LED:LED_0603_1608Metric -> LED_SMD:LED_0603_1608Metric
- J3: renamed from J2; footprint GSD090012SEU:AMPHENOL_GSD090012SEU -> Project_Library:AMPHENOL_GSD090012SEU
- R15: renamed from R27; footprint Resistor_SMD:R_0201_0603Metric -> Resistor_SMD:R_0805_2012Metric
- R16: renamed from R28; footprint Resistor_SMD:R_0201_0603Metric -> Resistor_SMD:R_0805_2012Metric
- R17: renamed from R21; footprint Resistor_SMD:R_0201_0603Metric -> Resistor_SMD:R_0805_2012Metric
- R20: renamed from R23; footprint Resistor_SMD:R_0201_0603Metric -> Resistor_SMD:R_0805_2012Metric
- R21: renamed from R24; footprint Resistor_SMD:R_0201_0603Metric -> Resistor_SMD:R_0805_2012Metric
- R22: renamed from R25; footprint Resistor_SMD:R_0201_0603Metric -> Resistor_SMD:R_0805_2012Metric
- U4: value CP2102N-Axx-xQFN20 -> CP2102N-A02-GQFN20
- U6: renamed from U5; footprint W25Q32JVSSIQ:SOIC127P790X216-8N -> Project_Library:SOIC127P790X216-8N
- renumbered C11 to C10, C14 to C12, C15 to C13, C13 to C14, C8 to C7, C12 to C9, D9 to D5, R18 to R11, R14 to R12, R17 to R13, R20 to R14, R19 to R18
Connections:
- net 3.3V: now also C10.1, C9.1, R11.1, U4.7 (VREGIN), C8.2, R19.2
- net BOOT: now also U3.8 (IO9); no longer U3.18 (IO0)
- net CS: now also U6.1 (~{CS})
- net CS_SD: now also J3.1 (CD/DAT3), U3.18 (IO0), R19.1; no longer U3.8 (IO9)
- net GND: now also C11.2, C8.1, U5.2 (GND)
- net RX_TX: now also U3.12 (TXD)
- net TX_RX: now also U3.11 (RXD)
- net USB_DN: now also U5.4 (I/O2); no longer U4.5 (D-)
- net USB_DP: now also U5.6 (I/O1); no longer U4.4 (D+)
- net VBUS: now also U5.5 (VBUS); no longer C10.1, C9.1, R11.1, U4.7 (VREGIN)
- net at R12.2, R13.1, U4.8 (VBUS): now also C11.1
- new net: U4.4 (D+), U5.1 (I/O1)
- new net: U4.5 (D-), U5.3 (I/O2)
Other:
- moved on the sheet: C10, C7, C9, R11

Commit message: Configured the layout editor.
Parts:
- D5: footprint SparkFun-LED:LED_0603_1608Metric -> LED_SMD:LED_0603_1608Metric
- U3: footprint Footprints:MODULE_ESP32-C3-WROOM-02-H4 -> Project_Library:MODULE_ESP32-C3-WROOM-02-H4
Changed lines of the file:
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@@
 			)
 		)
-		(property "Footprint" "Footprints:MODULE_ESP32-C3-WROOM-02-H4"
+		(property "Footprint" "Project_Library:MODULE_ESP32-C3-WROOM-02-H4"
 			(at 220.98 46.99 0)
 			(effects
@@
 			)
 		)
-		(property "Footprint" "SparkFun-LED:LED_0603_1608Metric"
+		(property "Footprint" "LED_SMD:LED_0603_1608Metric"
 			(at 128.27 107.95 0)
 			(effects
@@
 		)
 		(instances
-			(project "KLP-5e-ESP32-sensor-board-main_modifications"
+			(project "ESP32 sensor board"
 				(path "/16c571a0-8550-4f05-972c-22b0701cbf02/09ec4a32-ddff-43cd-8e21-9ef822101853"
 					(page "3")
@@
 		)
 		(instances
-			(project "KLP-5e-ESP32-sensor-board-main_modifications"
+			(project "ESP32 sensor board"
 				(path "/16c571a0-8550-4f05-972c-22b0701cbf02/09ec4a32-ddff-43cd-8e21-9ef822101853"
 					(page "4")
