File: KiCad project/ESP32 sensor board.kicad_pcb (KiCad board)
At the start: 4 copper layers, 89.5 x 52.8 mm, 87 parts, among them J1 USB_C_Receptacle, J2 JST_2mm_LiPo, J3 GSD090012SEU, J4 B4B-XH-AM, J6 Conn_01x05, Q1 TEMT6000X01, Q2 BC817, Q3 BC817, SW1 1101NE, SW2 1101NE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

Commit message: Optimisation complete.
Parts:
- removed R17, R21: 50, Resistor_SMD:R_0805_2012Metric
- U1: footprint Footprints:QFN50P400X400X100-21N -> Package_DFN_QFN:QFN-20-1EP_4x4mm_P0.5mm_EP2.5x2.5mm
- moved TP1 16.4 mm to (167.6, 99.9)
- moved R15 15.5 mm to (176.3, 89.5), turned to 90 degrees
- moved TP3 14.7 mm to (174.0, 89.2)
- moved R13 11.9 mm to (153.1, 103.0), turned to 0 degrees
- moved TP2 11.3 mm to (164.1, 99.9)
- moved TP5 10.9 mm to (159.8, 87.0)
- moved R3 10.8 mm to (136.7, 119.4), turned to -90 degrees
- moved R4 9.83 mm to (136.7, 114.3), turned to -90 degrees
- moved U4 9.08 mm to (142.7, 100.2), turned to 90 degrees
- moved C14 7.62 mm to (159.9, 91.2), turned to -90 degrees
- moved R11 7.32 mm to (145.2, 95.9), turned to -90 degrees
- moved D6 5.88 mm to (138.5, 93.0)
- moved R16 5.77 mm to (167.6, 96.6)
- moved R18 5.77 mm to (138.5, 98.0)
- moved R12 5.58 mm to (149.3, 104.1), turned to 0 degrees
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Connections:
- J3 pad 2: Net-(J3-CMD) -> /ESP32-C3-02/MOSI_DI
- J3 pad 5: Net-(J3-CLK) -> /ESP32-C3-02/SCLK
- R12 pad 1: /+5V_USB -> /VBUS
- R15 pad 1: Net-(J3-CMD) -> /ESP32-C3-02/MOSI_DI
- R15 pad 2: /ESP32-C3-02/MOSI_DI -> Net-(U3-IO7)
- R20 pad 2: Net-(U6-CLK) -> Net-(U3-IO6)
- U3 pad 5: /ESP32-C3-02/SCLK -> Net-(U3-IO6)
- U3 pad 6: /ESP32-C3-02/MOSI_DI -> Net-(U3-IO7)
- U5 pad 1: /ESP32-C3-02/USB_D+ -> /ESP32-C3-02/USB_D-
- U5 pad 3: /ESP32-C3-02/USB_D- -> /ESP32-C3-02/USB_D+
- U5 pad 5: /+5V_USB -> /VBUS
- U6 pad 5: Net-(U6-DI(IO0)) -> /ESP32-C3-02/MOSI_DI
- U6 pad 6: Net-(U6-CLK) -> /ESP32-C3-02/SCLK
Routing:
- net GND: track 200.5 -> 120.6 mm, vias 52 -> 53
- net /+5V_USB: track 35.8 -> 10.1 mm, vias 10 -> 11
- net 3.3V: track 90.5 -> 67.6 mm, vias 21 -> 26
- net /ESP32-C3-02/TX_RX: track 65.2 -> 87.5 mm
- net /ESP32-C3-02/DTS: track 13.1 -> 35.2 mm, vias 0 -> 2
- net /ESP32-C3-02/RTS: track 27.1 -> 49.0 mm, vias 2 -> 4
- net /USB_DP: track 29.7 -> 9.93 mm, vias 3 -> 1
- net /ESP32-C3-02/SCLK: track 43.6 -> 25.0 mm, vias 2 -> 0
- net /ESP32-C3-02/RX_TX: track 69.1 -> 87.4 mm
- net /ESP32-C3-02/GPIO19: track 131.0 -> 147.0 mm
- net /ESP32-C3-02/BOOT: track 69.6 -> 84.0 mm
- net /ESP32-C3-02/GPIO18: track 104.1 -> 89.9 mm
- net Net-(U4-~{TXT}/GPIO.2): track 19.3 -> 6.26 mm, vias 4 -> 0
- net Net-(U4-VBUS): track 25.8 -> 12.9 mm, vias 2 -> 0
- net Net-(U4-~{RXT}/GPIO.3): track 16.0 -> 3.52 mm, vias 4 -> 0
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- added copper zone on F.Cu, net +5V
- added copper zone on F.Cu, net /+5V_USB
- added copper zone on F.Cu, net /VBAT
- added copper zone on F.Cu, net /VBUS
- added copper zone on In2.Cu, net /VBUS
- added copper zone on F.Cu, net 3.3V
- added copper zone on F.Cu, net GND
Other:
- outline, holes or cut-outs redrawn
- board text added: "ESP32 C3"
- board text added: "Environment"
- board text added: "Sensor"
- board text removed: "ESP32 S3"
- board text removed: "Environment sensor"
- board text removed: "IO18"
- board text removed: "IO19"
- board text removed: "IO8"
