File: KiCad project/user_interface.kicad_sch (KiCad schematic)
At the start: 11 parts, among them J4 B4B-XH-AM, J6 Conn_01x05, Q2 BC817, Q3 BC817, SW1 1101NE, SW2 1101NE

Commit message: Completed schematic fixes and updates. Continuing with the layout for Prototype #2.
Parts:
- J4: footprint Project_Library:JST_B4B-XH-AM__LF__SN_ -> Footprints:JST_B4B-XH-AM__LF__SN_
- SW1, SW2: footprint TL3305AF260QG:SW_TL3305AF260QG -> Footprints:SW_TL3305AF260QG
Changed lines of the file:
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@@
 			"qYIEwNEuIr4VFAXA5HoUrkfh9D+pnEDbYjcEwCGF61G4HgXA5HoUrkfh9D+ZPCzUmuYDwCCF61G4"
 			"HgXA5HoUrkfh9D+gPCzUmuYDQM8uIr4VFAXA5HoUrkfh9D+vnEDbYjcEQC50y4zn9ATA5HoUrkfh"
-			"9D/f4AuTqYIEQMDODbdNwwTA5HoUrkfh9D+/zg23TcMEQODgC5OpggTA5A=="
+			"9D/f4AuTqYIEQMDODbdNwwTA5HoUrkfh9D+/zg23TcMEQODgC5OpggTA5AAAAAAAAAAAAAAAAAAA"
+			"AAAAAAAAAAAAAAAAAAAAAAAAAAAAAAAAAAAAAAAAAAAAAPzSIQEAAACebtIhAQAAAAAAAAAAAAAA"
+			"axAAAAAAAAADAAAACd7HPg5Pwv0Osi5BIF8HAAAAHSnbwP0Osi5BAAAAAAAAAAAAAAAAAAAAAAAA"
+			"AAAAAAAAAAAAAAAAAAAAAAAAAAAAAAAAAAAAAAAAAAAAAAAAAAAAAAAAAAAAAAAAAAAAAAAAAAAA"
+			"AAAAAAAAAAAAAAAAAAAAAAAAAAAAAAAAAAAAAAAAAAAAAAAAAAAAAAAAAAAAAAAAAAAAAAAAAAAA"
+			"AAAAAAAAAAAAAAAAAAAAAAAAAAAAAAAAAAAAAAAAAAAAAAAAAAAAAAAAAAAAAAAAAAAAAAAAAAAA"
+			"AAAAAAAAAAAAAAAAAAAAAAAAAAAAAAAAAAAAAAAAAAAAAAAAAAAAAAAAAAAAAAAAAAAAAAAAAAAA"
+			"AAAAAAAAAAAAAAAAAAAAAAAAAAAAAAAAAAAAAAAAAAAAAAAAAAAAAAAAAAAAAAAAAAAAAAAAAAAA"
+			"AAAAAAAAAAAAAAAAAAAAAAAAAAAAAAAAAAAAAAAAAAAAAAAAAAAAAAAAAAAAAAAAAAAAAAAAAAAA"
+			"AAAAAAAAAAAAAAAAAAAAAAAAAAAAAAAAAAAAAAAAAAAAAAAAAAAAAAAAAAAAAAAAAAAAAAAAAAAA"
+			"AAAAAAAAAAAAAAAAAAAAAAAAAAAAAAAAAAAAAAAAAAAAAAAAAAAAAAAAAAAAAAAAAAAAAAAAAAAA"
+			"AAAAAAAAAAAAAAAAAAAAAAAAAAAAAAAAAAAAAAAAAAAAAAAAAAAAAAAAAAAAAAAAAAAAAAAAAAAA"
+			"AAAAAAAAAAAAAAAAAAAAAAAAAAAAAAAAAAAAAAAAAAAAAAAAAAAAAAAAAAAAAAAAAAAAAAAAAAAA"
+			"AAAAAAAAAAAAAAAAAAAAAAAAAAAAAAAAAAAAAAAAAAAAAAAAAAAAAAAAAAAAAAAAAAAAAAAAAAAA"
+			"AAAAAAAAAAAAAAAAAAAAAAAAAAAAAAAAAAAAAAAAAAAAAAAAAAAAAAAAAAAAAAAAAAAAAAAAAAAA"
+			"AAAAAAAAAAAAAAAAAAAAAAAAAAAAAAAAAAAAAAAAAAAAAAAAAAAAAAAAAAAAAAAAAAAAAAAAAAAA"
+			"AAAAAAAAAAAAAAAAAAAAAAAAAAAAAAAAAAAAAAAAAAAAAAAAAAAAAAAAAAAAAAAAAAAAAAAAAAAA"
+			"AAAAAAAAAAAAAAAAAAAAAAAAAAAAAAAAAAAAAAAAAAAAAAAAAAAAAAAAAAAAAAAAAAAAAAAAAAAA"
+			"AAAAAAAAAAAAAAAAAAAAAAAAAAAAAAAAAAAAAAAAAAAAAAAAAAAAAAAAAA=="
 		)
 	)
@@
 			)
 		)
-		(property "Footprint" "TL3305AF260QG:SW_TL3305AF260QG"
+		(property "Footprint" "Footprints:SW_TL3305AF260QG"
 			(at 214.63 67.31 0)
 			(effects
@@
 			)
 		)
-		(property "Footprint" "Project_Library:JST_B4B-XH-AM__LF__SN_"
+		(property "Footprint" "Footprints:JST_B4B-XH-AM__LF__SN_"
 			(at 72.39 62.23 0)
 			(effects
@@
 			)
 		)
-		(property "Footprint" "TL3305AF260QG:SW_TL3305AF260QG"
+		(property "Footprint" "Footprints:SW_TL3305AF260QG"
 			(at 162.56 62.23 0)
 			(effects

Commit message: Set correct SW1 and SW2 symbols
Parts:
- SW1, SW2: footprint Footprints:SW_TL3305AF260QG -> USLPT2819DT2TR:SW_USLPT2819DT2TR; symbol TL3305AF260QG:TL3305AF260QG -> USLPT2819DT2TR:USLPT2819DT2TR; Check_prices https://www.snapeda.com/parts/TL3305AF260QG/E-Switch/view-p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 -> https://www.snapeda.com/parts/USLPT2819DT2TR/TE+Connectivit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; MANUFACTURER E-Switch -> TE CONNECTIVITY; MF E-Switch -> TE Connectivity; MP TL3305AF260QG -> USLPT2819DT2TR; PARTREV C -> P; Package SMD-4 E-Switch -> None; STANDARD Manufacturer recommendations -> Manufacturer Recommendations; SnapEDA_Link https://www.snapeda.com/parts/TL3305AF260QG/E-Switch/view-p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 -> https://www.snapeda.com/parts/USLPT2819DT2TR/TE+Connectivit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
Connections:
- net BOOT: now also SW1.3; no longer SW1.2
- net EN: now also SW2.3; no longer SW2.2
- net GND: now also SW1.2, SW2.2; no longer SW1.3, SW2.3
Changed lines of the file:
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@@
 	(wire
 		(pts
+			(xy 170.18 64.77) (xy 173.99 64.77)
+		)
+		(stroke
+			(width 0)
+			(type default)
+		)
+	)
+	(wire
+		(pts
 			(xy 157.48 111.76) (xy 158.75 111.76)
 		)
@@
 	(wire
 		(pts
+			(xy 170.18 59.69) (xy 175.26 59.69)
+		)
+		(stroke
+			(width 0)
+			(type default)
+		)
+	)
+	(wire
+		(pts
 			(xy 226.06 76.2) (xy 226.06 69.85)
 		)
@@
 	(wire
 		(pts
-			(xy 203.2 69.85) (xy 204.47 69.85)
+			(xy 203.2 69.85) (xy 207.01 69.85)
 		)
 		(stroke
@@
 	(wire
 		(pts
-			(xy 151.13 64.77) (xy 152.4 64.77)
+			(xy 222.25 69.85) (xy 226.06 69.85)
+		)
+		(stroke
+			(width 0)
+			(type default)
+		)
+	)
+	(wire
+		(pts
+			(xy 151.13 64.77) (xy 154.94 64.77)
 		)
 		(stroke
@@
 	(wire
 		(pts
-			(xy 151.13 59.69) (xy 152.4 59.69)
+			(xy 151.13 59.69) (xy 154.94 59.69)
 		)
 		(stroke
@@
 	(wire
 		(pts
-			(xy 203.2 64.77) (xy 204.47 64.77)
+			(xy 203.2 64.77) (xy 207.01 64.77)
 		)
 		(stroke
@@
 	(wire
 		(pts
-			(xy 224.79 64.77) (xy 227.33 64.77)
-		)
-		(stroke
-			(width 0)
-			(type default)
-		)
-	)
-	(wire
-		(pts
 			(xy 181.61 133.35) (xy 181.61 135.89)
 		)
@@
 	(wire
 		(pts
-			(xy 173.99 64.77) (xy 173.99 69.85)
-		)
-		(stroke
-			(width 0)
-			(type default)
-		)
-	)
-	(wire
-		(pts
-			(xy 227.33 57.15) (xy 227.33 64.77)
+			(xy 222.25 64.77) (xy 227.33 64.77)
 		)
 		(stroke
@@
 	(wire
 		(pts
-			(xy 172.72 59.69) (xy 175.26 59.69)
+			(xy 173.99 64.77) (xy 173.99 69.85)
 		)
 		(stroke
@@
 	(wire
 		(pts
-			(xy 226.06 69.85) (xy 224.79 69.85)
+			(xy 227.33 57.15) (xy 227.33 64.77)
 		)
 		(stroke
@@
 	(wire
 		(pts
-			(xy 172.72 64.77) (xy 173.99 64.77)
-		)
-		(stroke
-			(width 0)
-			(type default)
-		)
-	)
-	(wire
-		(pts
 			(xy 193.04 53.34) (xy 193.04 55.88)
 		)
@@
 	)
 	(symbol
-		(lib_id "TL3305AF260QG:TL3305AF260QG")
+		(lib_id "USLPT2819DT2TR:USLPT2819DT2TR")
 		(at 214.63 67.31 0)
 		(unit 1)
@@
 			)
 		)
-		(property "Footprint" "Footprints:SW_TL3305AF260QG"
+		(property "Footprint" "USLPT2819DT2TR:SW_USLPT2819DT2TR"
 			(at 214.63 67.31 0)
 			(effects
@@
 			)
 		)
-		(property "MF" "E-Switch"
+		(property "MF" "TE Connectivity"
 			(at 214.63 67.31 0)
 			(effects
@@
 			)
 		)
-		(property "Package" "SMD-4 E-Switch"
+		(property "Package" "None"
 			(at 214.63 67.31 0)
 			(effects
@@
 			)
 		)
-		(property "SnapEDA_Link" "https://www.snapeda.com/parts/TL3305AF260QG/E-Switch/view-part/?ref=snap"
+		(property "SnapEDA_Link" "https://www.snapeda.com/parts/USLPT2819DT2TR/TE+Connectivity+ALCOSWITCH+Switches/view-part/?ref=snap"
 			(at 214.63 67.31 0)
 			(effects
@@
 			)
 		)
-		(property "MP" "TL3305AF260QG"
+		(property "MP" "USLPT2819DT2TR"
 			(at 214.63 67.31 0)
 			(effects
@@
 			)
 		)
-		(property "Check_prices" "https://www.snapeda.com/parts/TL3305AF260QG/E-Switch/view-part/?ref=eda"
+		(property "Check_prices" "https://www.snapeda.com/parts/USLPT2819DT2TR/TE+Connectivity+ALCOSWITCH+Switches/view-part/?ref=eda"
 			(at 214.63 67.31 0)
 			(effects
@@
 			)
 		)
-		(property "STANDARD" "Manufacturer recommendations"
+		(property "STANDARD" "Manufacturer Recommendations"
 			(at 214.63 67.31 0)
 			(effects
@@
 			)
 		)
-		(property "PARTREV" "C"
+		(property "PARTREV" "P"
 			(at 214.63 67.31 0)
 			(effects
@@
 			)
 		)
-		(property "MANUFACTURER" "E-Switch"
+		(property "MANUFACTURER" "TE CONNECTIVITY"
 			(at 214.63 67.31 0)
 			(effects
@@
 	)
 	(symbol
-		(lib_id "TL3305AF260QG:TL3305AF260QG")
+		(lib_id "USLPT2819DT2TR:USLPT2819DT2TR")
 		(at 162.56 62.23 0)
 		(unit 1)
@@
 			)
 		)
-		(property "Footprint" "Footprints:SW_TL3305AF260QG"
+		(property "Footprint" "USLPT2819DT2TR:SW_USLPT2819DT2TR"
 			(at 162.56 62.23 0)
 			(effects
@@
 			)
 		)
-		(property "MF" "E-Switch"
+		(property "MF" "TE Connectivity"
 			(at 162.56 62.23 0)
 			(effects
@@
 			)
 		)
-		(property "Package" "SMD-4 E-Switch"
+		(property "Package" "None"
 			(at 162.56 62.23 0)
 			(effects
@@
 			)
 		)
-		(property "SnapEDA_Link" "https://www.snapeda.com/parts/TL3305AF260QG/E-Switch/view-part/?ref=snap"
+		(property "SnapEDA_Link" "https://www.snapeda.com/parts/USLPT2819DT2TR/TE+Connectivity+ALCOSWITCH+Switches/view-part/?ref=snap"
 			(at 162.56 62.23 0)
 			(effects
@@
 			)
 		)
-		(property "MP" "TL3305AF260QG"
+		(property "MP" "USLPT2819DT2TR"
 			(at 162.56 62.23 0)
 			(effects
@@
 			)
 		)
-		(property "Check_prices" "https://www.snapeda.com/parts/TL3305AF260QG/E-Switch/view-part/?ref=eda"
+		(property "Check_prices" "https://www.snapeda.com/parts/USLPT2819DT2TR/TE+Connectivity+ALCOSWITCH+Switches/view-part/?ref=eda"
 			(at 162.56 62.23 0)
 			(effects
@@
 			)
 		)
-		(property "STANDARD" "Manufacturer recommendations"
+		(property "STANDARD" "Manufacturer Recommendations"
 			(at 162.56 62.23 0)
 			(effects
@@
 			)
 		)
-		(property "PARTREV" "C"
+		(property "PARTREV" "P"
 			(at 162.56 62.23 0)
 			(effects
@@
 			)
 		)
-		(property "MANUFACTURER" "E-Switch"
+		(property "MANUFACTURER" "TE CONNECTIVITY"
 			(at 162.56 62.23 0)
 			(effects
